File: hardware/Version_02/Camera.brd (EAGLE design)
At the start: 44.4 x 42.9 mm, 40 parts, among them IC5 APX803, Q2 8MHz, U1 TPS61090RSAR, U2 MCP73831T-2ACI/OT, U3 ATMEGA328

Commit message: Latest version
Parts:
- moved GROUND_1 11.2 mm to (23.1, 11.3)
- moved SHUTTER 9.30 mm to (23.1, 14.1)
- moved ON/OFF 9.09 mm to (25.6, 14.1)
- moved TXO 4.01 mm to (25.6, 19.9)
- moved RXI 3.87 mm to (25.6, 17.1)
- moved DTR 2.55 mm to (23.1, 17.1)
- moved CAM_BOTTOM 2.54 mm to (19.0, 24.5)
- moved CAM_TOP 2.54 mm to (14.7, 24.5)
- moved GROUND_2 2.54 mm to (23.1, 20.0)
- moved C5 2.53 mm to (40.7, 23.4), turned to 90 degrees
- moved B1 1.80 mm to (14.3, 11.2)
- moved C9 1.56 mm to (11.5, 30.3), turned to 0 degrees
- moved C10 1.31 mm to (11.5, 28.3), turned to 0 degrees
- moved R16 1.05 mm to (11.5, 26.3), turned to 0 degrees
- moved R17 0.84 mm to (11.5, 24.2)
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Routing:
- net GND: track 0.00 -> 127.0 mm, vias 0 -> 11
- net 3.3V: track 0.00 -> 85.2 mm, vias 0 -> 1
- net 5.0V: track 0.00 -> 64.2 mm, vias 0 -> 2
- net A5/SCL: track 0.00 -> 59.5 mm, vias 0 -> 2
- net A4/SDA: track 0.00 -> 58.6 mm, vias 0 -> 2
- net VBAT: track 0.00 -> 43.2 mm, vias 0 -> 2
- net DTR: track 0.00 -> 20.7 mm, vias 0 -> 2
- net RXI: track 0.00 -> 19.4 mm, vias 0 -> 2
- net VDD1: track 0.00 -> 17.9 mm, vias 0 -> 1
- net D3: track 0.00 -> 17.1 mm, vias 0 -> 1
- net ENABLE: track 0.00 -> 16.8 mm, vias 0 -> 2
- net TXO: track 0.00 -> 15.7 mm, vias 0 -> 2
- net D4: track 0.00 -> 14.3 mm, vias 0 -> 1
- net !OLED_RST: track 0.00 -> 14.1 mm, vias 0 -> 2
- net N$3: track 0.00 -> 10.5 mm
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- added copper zone on layer 1, net GND
- added copper zone on layer 16, net GND
