File: hardware/Version_03/Camera.brd (EAGLE design)
At the start: 55.8 x 42.9 mm, 44 parts, among them IC5 APX803, Q2 8MHz, U1 TPS61090RSAR, U2 MCP73831T-2ACI/OT, U3 ATMEGA328, X1 52745-1490, X2 52745-1490, X3 52745-1490

Commit message: Version 3 for production
Parts:
- removed LCD1, LCD2: OLED 128x32, microbuilder:UG-2832HSWEG02_WRAPUNDER
- removed X1, X3: 52745-1490, con-molex:52745-1490
Connections:
- removed net N$38: LCD1.1, X1.14
- removed net N$39: LCD1.2, X1.13
- removed net N$40: LCD1.3, X1.12
- removed net N$41: LCD1.4, X1.11
- removed net N$42: LCD1.5, X1.10
- removed net N$43: LCD1.14, X1.1
- removed net N$44: LCD1.13, X1.2
- removed net N$45: LCD1.12, X1.3
- removed net N$46: LCD1.11, X1.4
- removed net N$47: LCD1.10, X1.5
- removed net N$48: LCD1.9, X1.6
- removed net N$49: LCD1.8, X1.7
- removed net N$50: LCD1.7, X1.8
- removed net N$51: LCD1.6, X1.9
- removed net N$52: LCD2.1, X3.1
- removed net N$53: LCD2.2, X3.2
- removed net N$54: LCD2.3, X3.3
- removed net N$55: LCD2.4, X3.4
- removed net N$56: LCD2.5, X3.5
- removed net N$57: LCD2.6, X3.6
- removed net N$58: LCD2.7, X3.7
- removed net N$59: LCD2.8, X3.8
- removed net N$60: LCD2.9, X3.9
- removed net N$61: LCD2.10, X3.10
- removed net N$62: LCD2.11, X3.11
- removed net N$63: LCD2.12, X3.12
- removed net N$64: LCD2.13, X3.13
- removed net N$65: LCD2.14, X3.14
Routing:
- net N$59: track 5.38 -> 0.00 mm, vias 1 -> 0
- net N$54: track 5.29 -> 0.00 mm, vias 1 -> 0
- net N$63: track 5.25 -> 0.00 mm, vias 1 -> 0
- net N$56: track 5.20 -> 0.00 mm, vias 1 -> 0
- net N$61: track 5.17 -> 0.00 mm, vias 1 -> 0
- net N$58: track 5.10 -> 0.00 mm, vias 1 -> 0
- net N$38: track 4.70 -> 0.00 mm
- net N$43: track 4.67 -> 0.00 mm
- net N$39: track 4.65 -> 0.00 mm
- net N$44: track 4.63 -> 0.00 mm
- net N$40: track 4.60 -> 0.00 mm
- net N$45: track 4.57 -> 0.00 mm
- net N$41: track 4.55 -> 0.00 mm
- net N$46: track 4.52 -> 0.00 mm
- net N$42: track 4.50 -> 0.00 mm
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Other:
- board size 55.8 x 42.9 mm -> 44.4 x 42.9 mm
