File: hardware/Version_03/Camera.sch (EAGLE design)
At the start: 44 parts, among them IC5 APX803, Q2 8MHz, U1 TPS61090RSAR, U2 MCP73831T-2ACI/OT, U3 ATMEGA328, X1 52745-1490, X2 52745-1490, X3 52745-1490

Commit message: Version 3 for production
Parts:
- removed LCD1, LCD2: OLED 128x32, microbuilder:DISP_OLED_UG-2832HSWEG02
- removed X1, X3: 52745-1490, con-molex:52745-1490
Connections:
- removed net N$38: LCD1.C2+, X1-14.S
- removed net N$39: LCD1.C2-, X1-13.S
- removed net N$40: LCD1.C1+, X1-12.S
- removed net N$41: LCD1.C1-, X1-11.S
- removed net N$42: LCD1.VBAT, X1-10.S
- removed net N$43: LCD1.VCC, X1-1.S
- removed net N$44: LCD1.VCOMH, X1-2.S
- removed net N$45: LCD1.IREF, X1-3.S
- removed net N$46: LCD1.SDA, X1-4.S
- removed net N$47: LCD1.SCL, X1-5.S
- removed net N$48: LCD1.RES#, X1-6.S
- removed net N$49: LCD1.VDD, X1-7.S
- removed net N$50: LCD1.VSS, X1-8.S
- removed net N$51: LCD1.VBREF, X1-9.S
- removed net N$52: LCD2.C2+, X3-1.S
- removed net N$53: LCD2.C2-, X3-2.S
- removed net N$54: LCD2.C1+, X3-3.S
- removed net N$55: LCD2.C1-, X3-4.S
- removed net N$56: LCD2.VBAT, X3-5.S
- removed net N$57: LCD2.VBREF, X3-6.S
- removed net N$58: LCD2.VSS, X3-7.S
- removed net N$59: LCD2.VDD, X3-8.S
- removed net N$60: LCD2.RES#, X3-9.S
- removed net N$61: LCD2.SCL, X3-10.S
- removed net N$62: LCD2.SDA, X3-11.S
- removed net N$63: LCD2.IREF, X3-12.S
- removed net N$64: LCD2.VCOMH, X3-13.S
- removed net N$65: LCD2.VCC, X3-14.S
Other:
- note removed: "OLED CONNECTOR"
